File: schematics/synthiota1/synthiota1.kicad_sch (KiCad schematic)
At the start: 111 parts, among them IC1 H11L1, J1 PJ-320A-4P DIP, J2 PJ-320A-4P DIP, SW1 SW_Push, SW2 SW_Push, SW3 SW_Push, U1 Pico, U2 74HC4051, U3 MPR121QR2, U4 MPR121QR2

Commit message: pcb cleanup
Parts:
- added C33: 100n, Capacitor_SMD:C_0603_1608Metric, symbol Device:C
- renumbered C100 to C28, C104 to C29, C103 to C30, C101 to C31, C102 to C32, D100 to D1, U1 to MODULE1, MODULE1 to MODULE2, R17 to R1, R18 to R2, R20 to R3, R19 to R4, R24 to R5, R21 to R6, IC1 to U1
Connections:
- net +3V3: now also C33.1
- net GND: now also C33.2
Other:
- moved on the sheet: LED25, LED26, LED27

Commit message: lcsc part nums for everything because jlc sucks now, pcb cleanup
Parts:
- C1, C10, C11, C12, C13, C14, C15, C16, C17, C18, C19, C2, C20, C21, C22, C23, C24, C25, C26, C27, C28, C29, C3, C30, C31, C32, C33, C4, C5, C6, C7, C8, C9: LCSC Part (none) -> C1590
- D1: LCSC Part (none) -> C81598
- LED10, LED11, LED12, LED13, LED14, LED15, LED16, LED17, LED18, LED19, LED2, LED20, LED21, LED22, LED23, LED24, LED25, LED26, LED27, LED3, LED4, LED5, LED6, LED7, LED8, LED9: LCSC Part (none) -> C5149201
- R1: LCSC Part (none) -> C22859
- R2: LCSC Part (none) -> C23140
- R22, R23, R4: LCSC Part (none) -> C23162
- R3: LCSC Part (none) -> C8218
- R5, R6: LCSC Part (none) -> C23242
- U1: LCSC Part (none) -> C78589
- U2: LCSC Part (none) -> C2943297

Commit message: added up/dn buttons! and more pcb tweaks
Parts:
- added TP17, TP18: Capacitive_Button, todbot_stuff:Pad-CapTouch-8mm-roundrect, symbol todbot_stuff:Capacitive_Button
Connections:
- net at U4.15 (LED3/ELE7): now also TP18.1 (A)
- net at U4.16 (LED4/ELE8): now also TP17.1 (A)
- no-connect marks 38 -> 36
Other:
- moved on the sheet: SLIDER1
Changed lines of the file:
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@@
 	)
 	(no_connect
-		(at 146.05 172.72)
-	)
-	(no_connect
 		(at 71.12 36.83)
 	)
@@
 	)
 	(no_connect
-		(at 146.05 175.26)
-	)
-	(no_connect
 		(at 25.4 24.13)
 	)
@@
 	(wire
 		(pts
-			(xy 138.43 172.72) (xy 146.05 172.72)
-		)
-		(stroke
-			(width 0)
-			(type default)
-		)
-	)
-	(wire
-		(pts
 			(xy 389.89 162.56) (xy 389.89 134.62)
 		)
@@
 	(wire
 		(pts
+			(xy 172.72 193.04) (xy 172.72 182.88)
+		)
+		(stroke
+			(width 0)
+			(type default)
+		)
+	)
+	(wire
+		(pts
 			(xy 85.09 223.52) (xy 85.09 224.79)
 		)
@@
 	(wire
 		(pts
-			(xy 138.43 175.26) (xy 146.05 175.26)
+			(xy 138.43 175.26) (xy 154.94 175.26)
 		)
 		(stroke
@@
 	(wire
 		(pts
-			(xy 138.43 177.8) (xy 171.45 177.8)
+			(xy 138.43 177.8) (xy 173.99 177.8)
 		)
 		(stroke
@@
 	(wire
 		(pts
-			(xy 171.45 167.64) (xy 173.99 167.64)
-		)
-		(stroke
-			(width 0)
-			(type default)
-		)
-	)
-	(wire
-		(pts
 			(xy 326.39 204.47) (xy 323.85 204.47)
 		)
@@
 	(wire
 		(pts
-			(xy 138.43 182.88) (xy 173.99 182.88)
+			(xy 172.72 193.04) (xy 173.99 193.04)
 		)
 		(stroke
@@
 	(wire
 		(pts
+			(xy 138.43 172.72) (xy 167.64 172.72)
+		)
+		(stroke
+			(width 0)
+			(type default)
+		)
+	)
+	(wire
+		(pts
 			(xy 402.59 240.03) (xy 400.05 240.03)
 		)
@@
 	(wire
 		(pts
-			(xy 173.99 180.34) (xy 173.99 175.26)
+			(xy 173.99 180.34) (xy 173.99 185.42)
 		)
 		(stroke
@@
 	(wire
 		(pts
-			(xy 171.45 177.8) (xy 171.45 167.64)
+			(xy 172.72 182.88) (xy 138.43 182.88)
 		)
 		(stroke
@@
 	(symbol
 		(lib_id "todbot_eagle2023:TouchSlider-3sectors")
-		(at 184.15 175.26 0)
+		(at 184.15 185.42 0)
 		(mirror x)
 		(unit 1)
@@
 		(dnp no)
 		(property "Reference" "SLIDER1"
-			(at 187.96 176.53 0)
+			(at 187.96 186.69 0)
 			(effects
 				(font
@@
 		)
 		(property "Value" "~"
-			(at 179.07 162.56 0)
+			(at 179.07 172.72 0)
 			(effects
 				(font
@@
 		)
 		(property "Footprint" "todbot_stuff:TouchSlider3_50x8mm_ti"
-			(at 184.15 175.26 0)
+			(at 184.15 185.42 0)
 			(effects
 				(font
@@
 		)
 		(property "Datasheet" ""
-			(at 184.15 175.26 0)
+			(at 184.15 185.42 0)
 			(effects
 				(font
@@
 		)
 		(property "Description" ""
-			(at 184.15 175.26 0)
+			(at 184.15 185.42 0)
 			(effects
 				(font
@@
 		)
 		(property "Display" ""
-			(at 184.15 175.26 0)
+			(at 184.15 185.42 0)
 			(effects
 				(font
@@
 		)
 		(property "Manufacturer" ""
-			(at 184.15 175.26 0)
+			(at 184.15 185.42 0)
 			(effects
 				(font
@@
 		)
 		(property "Part Number" ""
-			(at 184.15 175.26 0)
+			(at 184.15 185.42 0)
 			(effects
 				(font
@@
 		)
 		(property "Specifications" ""
-			(at 184.15 175.26 0)
+			(at 184.15 185.42 0)
 			(effects
 				(font
@@
 	)
 	(symbol
+		(lib_id "todbot_stuff:Capacitive_Button")
+		(at 154.94 175.26 270)
+		(unit 1)
+		(exclude_from_sim no)
+		(in_bom yes)
+		(on_board yes)
+		(dnp no)
+		(fields_autoplaced yes)
+		(property "Reference" "TP17"
+			(at 161.29 173.9899 90)
+			(effects
+				(font
+					(size 1.27 1.27)
+				)
+				(justify left)
+			)
+		)
+		(property "Value" "Capacitive_Button"
+			(at 161.29 176.5299 90)
+			(effects
+				(font
+					(size 1.27 1.27)
+				)
+				(justify left)
+			)
+		)
+		(property "Footprint" "todbot_stuff:Pad-CapTouch-8mm-roundrect"
+			(at 147.32 175.26 0)
+			(effects
+				(font
+					(size 1.27 1.27)
+				)
+				(hide yes)
+			)
+		)
+		(property "Datasheet" "~"
+			(at 144.78 175.26 0)
+			(effects
+				(font
+					(size 1.27 1.27)
+				)
+				(hide yes)
+			)
+		)
+		(property "Description" "Capacitive touch pad"
+			(at 154.94 175.26 0)
+			(effects
+				(font
+					(size 1.27 1.27)
+				)
+				(hide yes)
+			)
+		)
+		(pin "1"
+		)
+		(instances
+			(project "synthiota1"
+				(path "/91d40f58-a363-48c7-98aa-eb2459062304"
+					(reference "TP17")
+					(unit 1)
+				)
+			)
+		)
+	)
+	(symbol
 		(lib_id "PCM_marbastlib-various:SK6812MINI-E")
 		(at 280.67 173.99 0)
@@
 					(unit 1)
 				)
+			)
+		)
+	)
+	(symbol
+		(lib_id "todbot_stuff:Capacitive_Button")
+		(at 167.64 172.72 270)
+		(unit 1)
+		(exclude_from_sim no)
+		(in_bom yes)
+		(on_board yes)
+		(dnp no)
+		(fields_autoplaced yes)
+		(property "Reference" "TP18"
+			(at 173.99 171.4499 90)
+			(effects
+				(font
+					(size 1.27 1.27)
+				)
+				(justify left)
+			)
+		)
+		(property "Value" "Capacitive_Button"
+			(at 173.99 173.9899 90)
+			(effects
+				(font
+					(size 1.27 1.27)
+				)
+				(justify left)
+			)
+		)
+		(property "Footprint" "todbot_stuff:Pad-CapTouch-8mm-roundrect"
+			(at 160.02 172.72 0)
+			(effects
+				(font
+					(size 1.27 1.27)
+				)
+				(hide yes)
+			)
+		)
+		(property "Datasheet" "~"
+			(at 157.48 172.72 0)
+			(effects
+				(font
+					(size 1.27 1.27)
+				)
+				(hide yes)
+			)
+		)
+		(property "Description" "Capacitive touch pad"
+			(at 167.64 172.72 0)
+			(effects
+				(font
+					(size 1.27 1.27)
+				)
+				(hide yes)
+			)
+		)
+		(pin "1"
+		)
+		(instances
+			(project ""
+				(path "/91d40f58-a363-48c7-98aa-eb2459062304"
+					(reference "TP18")
+					(unit 1)
+				)

Commit message: rotary encoder instead
Parts:
- removed SW1, SW2, SW3: SW_Push, Button_Switch_THT:SW_PUSH_6mm_H4.3mm, symbol Switch:SW_Push
- added SW1: RotaryEncoder_Switch_MP, PCM_marbastlib-various:ROT_Alps_EC11E-Switch, symbol Device:RotaryEncoder_Switch_MP
Connections:
- net GND: now also SW1.C, SW1.S2
- net SWA: now also MODULE1.32 (GPIO27_ADC1), SW1.A; no longer MODULE1.34 (GPIO28_ADC2)
- net SWB: now also MODULE1.34 (GPIO28_ADC2), SW1.B; no longer MODULE1.32 (GPIO27_ADC1)
- net SWC: now also SW1.S1
- no-connect marks 36 -> 37
