File: schematics/synthiota1/synthiota1.kicad_pcb (KiCad board)
At the start: 2 copper layers, 177.8 x 114.3 mm, 113 parts, among them J1 PJ-320A-4P DIP, J2 PJ-320A-4P DIP, SW1 RotaryEncoder_Switch_MP, U1 H11L1, U2 74HC4051, U3 MPR121QR2, U4 MPR121QR2

Commit message: as submitted to jlcpcb fab
Parts:
- removed the U1 at (106.4, 31.0) (x2)
- added U1: H11L1, easyeda2kicad:SMD-6_L7.3-W6.5-P2.54-LS10.2-BL, B.Cu at (106.4, 31.0)
