File: schematics/synthiota1/synthiota1.kicad_pcb (KiCad board)
At the start: 2 copper layers, 177.8 x 114.3 mm, 112 parts, among them J1 PJ-320A-4P DIP, J2 PJ-320A-4P DIP, SW1 RotaryEncoder_Switch_MP, U1 H11L1, U2 74HC4051, U3 MPR121QR2, U4 MPR121QR2

Commit message: assembly directions start
Parts:
- moved TP18 3.40 mm to (114.0, 82.4)
- moved TP17 2.60 mm to (98.0, 82.4)
Routing:
- net Net-(TP17-A): track 18.5 -> 13.4 mm
- net Net-(TP18-A): track 26.8 -> 24.3 mm
Changed lines of the file:
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@@
 	(footprint "todbot_stuff:Pad-CapTouch-8mm-roundrect"
 		(layer "F.Cu")
-		(at 95.4 82.4)
+		(at 98 82.4)
 		(descr "<h3>Conductive Button</h3>\n<p>Used with rubber key pads on the <a href=\"https://www.sparkfun.com/products/retired/8602\">Nordic Key FOB</a>. This one was designed and proven to work with the <a href=\"https://www.sparkfun.com/products/retired/9377\">PolyCase Key FOB enclosures</a>.</p>")
 		(property "Reference" "TP17"
@@
 	(footprint "todbot_stuff:Pad-CapTouch-8mm-roundrect"
 		(layer "F.Cu")
-		(at 117.4 82.4)
+		(at 114 82.4)
 		(descr "<h3>Conductive Button</h3>\n<p>Used with rubber key pads on the <a href=\"https://www.sparkfun.com/products/retired/8602\">Nordic Key FOB</a>. This one was designed and proven to work with the <a href=\"https://www.sparkfun.com/products/retired/9377\">PolyCase Key FOB enclosures</a>.</p>")
 		(property "Reference" "TP18"
@@
 	)
 	(gr_arc
-		(start 97.4 78.9)
-		(mid 98.46066 79.33934)
-		(end 98.9 80.4)
+		(start 100 78.9)
+		(mid 101.06066 79.33934)
+		(end 101.5 80.4)
 		(stroke
 			(width 0.1)
@@
 	)
 	(gr_arc
-		(start 91.9 80.4)
-		(mid 92.33934 79.33934)
-		(end 93.4 78.9)
+		(start 94.5 80.4)
+		(mid 94.93934 79.33934)
+		(end 96 78.9)
 		(stroke
 			(width 0.1)
@@
 	)
 	(gr_line
-		(start 91.9 84.4)
-		(end 91.9 80.4)
+		(start 94.5 84.4)
+		(end 94.5 80.4)
 		(stroke
 			(width 0.1)
@@
 	)
 	(gr_line
-		(start 113.9 84.4)
-		(end 113.9 80.4)
+		(start 110.5 84.4)
+		(end 110.5 80.4)
 		(stroke
 			(width 0.1)
@@
 	)
 	(gr_arc
-		(start 113.9 80.4)
-		(mid 114.33934 79.33934)
-		(end 115.4 78.9)
+		(start 110.5 80.4)
+		(mid 110.93934 79.33934)
+		(end 112 78.9)
 		(stroke
 			(width 0.1)
@@
 	)
 	(gr_line
-		(start 97.4 85.9)
-		(end 93.4 85.9)
+		(start 100 85.9)
+		(end 96 85.9)
 		(stroke
 			(width 0.1)
@@
 	)
 	(gr_line
-		(start 115.4 78.9)
-		(end 119.4 78.9)
+		(start 112 78.9)
+		(end 116 78.9)
 		(stroke
 			(width 0.1)
@@
 	)
 	(gr_line
-		(start 98.9 80.4)
-		(end 98.9 84.4)
+		(start 101.5 80.4)
+		(end 101.5 84.4)
 		(stroke
 			(width 0.1)
@@
 	)
 	(gr_line
-		(start 120.9 80.4)
-		(end 120.9 84.4)
+		(start 117.5 80.4)
+		(end 117.5 84.4)
 		(stroke
 			(width 0.1)
@@
 	)
 	(gr_arc
-		(start 115.4 85.9)
-		(mid 114.33934 85.46066)
-		(end 113.9 84.4)
+		(start 112 85.9)
+		(mid 110.93934 85.46066)
+		(end 110.5 84.4)
 		(stroke
 			(width 0.1)
@@
 	)
 	(gr_arc
-		(start 119.4 78.9)
-		(mid 120.46066 79.33934)
-		(end 120.9 80.4)
+		(start 116 78.9)
+		(mid 117.06066 79.33934)
+		(end 117.5 80.4)
 		(stroke
 			(width 0.1)
@@
 	)
 	(gr_arc
-		(start 120.9 84.4)
-		(mid 120.46066 85.46066)
-		(end 119.4 85.9)
+		(start 117.5 84.4)
+		(mid 117.06066 85.46066)
+		(end 116 85.9)
 		(stroke
 			(width 0.1)
@@
 	)
 	(gr_line
-		(start 93.4 78.9)
-		(end 97.4 78.9)
+		(start 96 78.9)
+		(end 100 78.9)
 		(stroke
 			(width 0.1)
@@
 	)
 	(gr_line
-		(start 119.4 85.9)
-		(end 115.4 85.9)
+		(start 116 85.9)
+		(end 112 85.9)
 		(stroke
 			(width 0.1)
@@
 	)
 	(gr_arc
-		(start 93.4 85.9)
-		(mid 92.33934 85.46066)
-		(end 91.9 84.4)
+		(start 96 85.9)
+		(mid 94.93934 85.46066)
+		(end 94.5 84.4)
 		(stroke
 			(width 0.1)
@@
 	)
 	(gr_arc
-		(start 98.9 84.4)
-		(mid 98.46066 85.46066)
-		(end 97.4 85.9)
+		(start 101.5 84.4)
+		(mid 101.06066 85.46066)
+		(end 100 85.9)
 		(stroke
 			(width 0.1)
@@
 	)
 	(gr_text "↑"
-		(at 95.4 81.4 0)
+		(at 98 82 0)
 		(layer "F.SilkS")
 		(effects
@@
 				(bold yes)
 			)
-			(justify top)
 		)
 	)
@@
 	)
 	(gr_text "↓"
-		(at 117.4 82.4 0)
+		(at 114 82.4 0)
 		(layer "F.SilkS")
 		(effects
@@
 	)
 	(segment
-		(start 92.4 87.9)
-		(end 92.4 82.9)
+		(start 98 87.9)
+		(end 98 82.4)
 		(width 0.17)
 		(layer "F.Cu")
@@
 	)
 	(via
-		(at 92.4 87.9)
+		(at 98 87.9)
 		(size 0.6)
 		(drill 0.3)
@@
 	)
 	(segment
-		(start 92.4 87.9)
-		(end 101.9 87.9)
-		(width 0.17)
-		(layer "B.Cu")
-		(net 148)
-	)
-	(segment
 		(start 101.9 87.9)
 		(end 104 85.8)
@@
 	)
 	(segment
-		(start 115.9 82.4)
-		(end 118.4 82.4)
+		(start 98 87.9)
+		(end 101.9 87.9)
 		(width 0.17)
-		(layer "F.Cu")
-		(net 149)
+		(layer "B.Cu")
+		(net 148)
 	)
 	(segment
-		(start 108.4 89.9)
-		(end 115.9 82.4)
+		(start 108.4 94.4)
+		(end 108.4 89.9)
 		(width 0.17)
 		(layer "F.Cu")
@@
 	)
 	(segment
-		(start 108.4 94.4)
-		(end 108.4 89.9)
+		(start 108.4 89.9)
+		(end 115.9 82.4)
 		(width 0.17)
 		(layer "F.Cu")
